File: pcb/darkroom-timer/logic_shifter.kicad_sch (KiCad schematic)
At the start: 3 parts, among them Q1 BSS138

Commit message: PCB Ready
Parts:
- Q1: Placement Required -> (none)
- R1, R2: footprint Resistor_SMD:R_0201_0603Metric -> Resistor_SMD:R_0805_2012Metric; Placement Required -> (none)
Changed lines of the file:
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@@
-			)
-		)
-		(property "Placement" "Required"
-			(at 133.35 105.41 90)
-			(effects
-				(font
-					(size 1.27 1.27)
-				)
-				(hide yes)
 			)
 		)
@@
 			)
 		)
-		(property "Footprint" "Resistor_SMD:R_0201_0603Metric"
+		(property "Footprint" "Resistor_SMD:R_0805_2012Metric"
 			(at 118.872 91.44 90)
 			(effects
@@
 		)
 		(property "InvenTree Part #" "96"
-			(at 120.65 91.44 0)
-			(effects
-				(font
-					(size 1.27 1.27)
-				)
-				(hide yes)
-			)
-		)
-		(property "Placement" "Required"
 			(at 120.65 91.44 0)
 			(effects
@@
 			)
 		)
-		(property "Footprint" "Resistor_SMD:R_0201_0603Metric"
+		(property "Footprint" "Resistor_SMD:R_0805_2012Metric"
 			(at 144.272 91.44 90)
 			(effects
@@
 			(at 146.05 91.44 0)
 			(effects
-				(font
-					(size 1.27 1.27)
-				)
-				(hide yes)
-			)
-		)
-		(property "Placement" "Required"
-			(at 146.05 91.44 0)
-			(effects
