File: pcb/darkroom-timer/sd.kicad_sch (KiCad schematic)
At the start: 1 part, among them J1 Micro_SD_Card_Det2

Commit message: PCB Ready
Parts:
- J1: InvenTree Part # (none) -> 736; Placement Required -> (none)
Connections:
- no-connect marks 0 -> 4
Changed lines of the file:
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@@
 	(generator_version "9.0")
 	(paper "A4")
+	(no_connect
+		(at 125.73 87.63)
+	)
+	(no_connect
+		(at 125.73 107.95)
+	)
+	(no_connect
+		(at 125.73 105.41)
+	)
+	(no_connect
+		(at 125.73 110.49)
+	)
 	(hierarchical_label "CLK"
 		(shape input)
@@
 	)
 	(hierarchical_label "DOUT"
-		(shape input)
+		(shape output)
 		(at 125.73 102.87 180)
 		(effects
@@
 			)
 		)
-		(property "Placement" "Required"
+		(property "InvenTree Part #" "736"
 			(at 148.59 97.79 0)
 			(effects
