File: pcb/darkroom-timer/ssd.kicad_sch (KiCad schematic)
At the start: 4 parts, among them U1 MAX7221xWG

Commit message: PCB Ready
Parts:
- added C4: 0.1uF, Capacitor_SMD:C_0805_2012Metric, symbol Device:C
- JP2: footprint PCM_SparkFun-Jumper:Jumper_2_NO -> Jumper:SolderJumper-2_P1.3mm_Open_Pad1.0x1.5mm; Placement Required -> (none)
- RV1: footprint Potentiometer_THT:Potentiometer_ACP_CA6-H2,5_Horizontal -> Frank:RKT6V; InvenTree Part # (none) -> 587; Placement Required -> (none)
- SSD1, U1: Placement Required -> (none)
Connections:
- net +5V: now also C4.1
- net GND: now also C4.2
- no-connect marks 0 -> 5
Changed lines of the file:
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@@
 	(generator_version "9.0")
 	(paper "A4")
+	(junction
+		(at 120.65 66.04)
+		(diameter 0)
+		(color 0 0 0 0)
+	)
+	(no_connect
+		(at 130.81 115.57)
+	)
+	(no_connect
+		(at 130.81 118.11)
+	)
+	(no_connect
+		(at 130.81 110.49)
+	)
+	(no_connect
+		(at 130.81 113.03)
+	)
+	(no_connect
+		(at 130.81 120.65)
+	)
 	(wire
 		(pts
@@
 	(wire
 		(pts
+			(xy 120.65 60.96) (xy 120.65 66.04)
+		)
+		(stroke
+			(width 0)
+			(type default)
+		)
+	)
+	(wire
+		(pts
 			(xy 200.66 102.87) (xy 200.66 90.17)
 		)
@@
 		(pts
 			(xy 130.81 87.63) (xy 140.97 87.63)
+		)
+		(stroke
+			(width 0)
+			(type default)
+		)
+	)
+	(wire
+		(pts
+			(xy 120.65 66.04) (xy 120.65 74.93)
 		)
 		(stroke
@@
 			)
 		)
-		(property "Footprint" "PCM_SparkFun-Jumper:Jumper_2_NO"
+		(property "Footprint" "Jumper:SolderJumper-2_P1.3mm_Open_Pad1.0x1.5mm"
 			(at 101.6 88.9 0)
 			(effects
@@
 		(property "Description" "Jumper, 2-pole, open"
 			(at 101.6 88.9 0)
-			(effects
-				(font
-					(size 1.27 1.27)
-				)
-				(hide yes)
-			)
-		)
-		(property "Placement" "Required"
-			(at 101.6 88.9 90)
 			(effects
 				(font
@@
 	(symbol
 		(lib_id "power:+5V")
-		(at 120.65 74.93 0)
+		(at 120.65 60.96 0)
 		(unit 1)
 		(exclude_from_sim no)
@@
 		(fields_autoplaced yes)
 		(property "Reference" "#PWR05"
-			(at 120.65 78.74 0)
+			(at 120.65 64.77 0)
 			(effects
 				(font
@@
 		)
 		(property "Value" "+5V"
-			(at 120.65 69.85 0)
+			(at 120.65 55.88 0)
 			(effects
 				(font
@@
 		)
 		(property "Footprint" ""
-			(at 120.65 74.93 0)
+			(at 120.65 60.96 0)
 			(effects
 				(font
@@
 		)
 		(property "Datasheet" ""
-			(at 120.65 74.93 0)
+			(at 120.65 60.96 0)
 			(effects
 				(font
@@
 		)
 		(property "Description" "Power symbol creates a global label with name \"+5V\""
-			(at 120.65 74.93 0)
+			(at 120.65 60.96 0)
 			(effects
 				(font
@@
 				(path "/c97b450d-2c45-46f5-9f2c-8311aa9564ad/596c817a-8203-40ab-ad65-e9d64764bfd4"
 					(reference "#PWR05")
+					(unit 1)
+				)
+			)
+		)
+	)
+	(symbol
+		(lib_id "Device:C")
+		(at 124.46 66.04 90)
+		(unit 1)
+		(exclude_from_sim no)
+		(in_bom yes)
+		(on_board yes)
+		(dnp no)
+		(fields_autoplaced yes)
+		(property "Reference" "C4"
+			(at 124.46 58.42 90)
+			(effects
+				(font
+					(size 1.27 1.27)
+				)
+			)
+		)
+		(property "Value" "0.1uF"
+			(at 124.46 60.96 90)
+			(effects
+				(font
+					(size 1.27 1.27)
+				)
+			)
+		)
+		(property "Footprint" "Capacitor_SMD:C_0805_2012Metric"
+			(at 128.27 65.0748 0)
+			(effects
+				(font
+					(size 1.27 1.27)
+				)
+				(hide yes)
+			)
+		)
+		(property "Datasheet" "~"
+			(at 124.46 66.04 0)
+			(effects
+				(font
+					(size 1.27 1.27)
+				)
+				(hide yes)
+			)
+		)
+		(property "Description" "Unpolarized capacitor"
+			(at 124.46 66.04 0)
+			(effects
+				(font
+					(size 1.27 1.27)
+				)
+				(hide yes)
+			)
+		)
+		(property "InvenTree Part #" "742"
+			(at 124.46 66.04 90)
+			(effects
+				(font
+					(size 1.27 1.27)
+				)
+				(hide yes)
+			)
+		)
+		(pin "2"
+		)
+		(pin "1"
+		)
+		(instances
+			(project "darkroom-timer"
+				(path "/c97b450d-2c45-46f5-9f2c-8311aa9564ad/596c817a-8203-40ab-ad65-e9d64764bfd4"
+					(reference "C4")
 					(unit 1)
 				)
@@
 	)
 	(symbol
+		(lib_id "power:GND")
+		(at 128.27 66.04 90)
+		(unit 1)
+		(exclude_from_sim no)
+		(in_bom yes)
+		(on_board yes)
+		(dnp no)
+		(fields_autoplaced yes)
+		(property "Reference" "#PWR058"
+			(at 134.62 66.04 0)
+			(effects
+				(font
+					(size 1.27 1.27)
+				)
+				(hide yes)
+			)
+		)
+		(property "Value" "GND"
+			(at 132.08 66.0399 90)
+			(effects
+				(font
+					(size 1.27 1.27)
+				)
+				(justify right)
+			)
+		)
+		(property "Footprint" ""
+			(at 128.27 66.04 0)
+			(effects
+				(font
+					(size 1.27 1.27)
+				)
+				(hide yes)
+			)
+		)
+		(property "Datasheet" ""
+			(at 128.27 66.04 0)
+			(effects
+				(font
+					(size 1.27 1.27)
+				)
+				(hide yes)
+			)
+		)
+		(property "Description" "Power symbol creates a global label with name \"GND\" , ground"
+			(at 128.27 66.04 0)
+			(effects
+				(font
+					(size 1.27 1.27)
+				)
+				(hide yes)
+			)
+		)
+		(pin "1"
+		)
+		(instances
+			(project ""
+				(path "/c97b450d-2c45-46f5-9f2c-8311aa9564ad/596c817a-8203-40ab-ad65-e9d64764bfd4"
+					(reference "#PWR058")
+					(unit 1)
+				)
+			)
+		)
+	)
+	(symbol
 		(lib_id "Display_Character:CC56-12EWA")
 		(at 168.91 87.63 0)
@@
 		)
 		(property "InvenTree Part #" "731"
-			(at 168.91 87.63 0)
-			(effects
-				(font
-					(size 1.27 1.27)
-				)
-				(hide yes)
-			)
-		)
-		(property "Placement" "Required"
 			(at 168.91 87.63 0)
 			(effects
@@
 			)
 		)
-		(property "Footprint" "Potentiometer_THT:Potentiometer_ACP_CA6-H2,5_Horizontal"
+		(property "Footprint" "Frank:RKT6V"
 			(at 101.6 80.01 0)
 			(effects
@@
 			)
 		)
-		(property "Placement" "Required"
+		(property "InvenTree Part #" "587"
 			(at 101.6 80.01 0)
 			(effects
@@
 			(at 120.65 100.33 0)
 			(effects
-				(font
-					(size 1.27 1.27)
-				)
-				(hide yes)
-			)
-		)
-		(property "Placement" "Required"
-			(at 120.65 100.33 0)
-			(effects
