File: pcb/darkroom-timer/uC.kicad_sch (KiCad schematic)
At the start: 4 parts

Commit message: PCB Ready
Parts:
- A1: footprint Module:RaspberryPi_Pico_Common_SMD -> Module:RaspberryPi_Pico_SMD_HandSolder; Placement Required -> (none)
- JP1: footprint PCM_SparkFun-Jumper:Jumper_2_NC_Trace -> Jumper:SolderJumper-2_P1.3mm_Bridged_Pad1.0x1.5mm; Placement Required -> (none)
- JP3: footprint PCM_SparkFun-Jumper:Jumper_2_NO -> Jumper:SolderJumper-2_P1.3mm_Open_Pad1.0x1.5mm; Placement Required -> (none)
- TP3: Placement Required -> (none)
Connections:
- net L_B: now also A1.9 (GPIO6); no longer A1.11 (GPIO8)
- net L_G: now also A1.7 (GPIO5); no longer A1.10 (GPIO7)
- net L_R: now also A1.6 (GPIO4); no longer A1.9 (GPIO6)
- net BUZZER: now reaches A1.29 (GPIO22)
- net BTN 1 renamed DI_PL
- net BTN 2 renamed DI_IN
- net BTN 3 renamed EPD_BUSY
- net BTN 4 renamed EPD_CS
- net BTN 5 renamed EPD_DC
- net BTN 6 renamed EPD_RES
- net RELAY renamed DI_CLK
- new net REL_ENLR: A1.11 (GPIO8)
- new net REL_SAFE: A1.10 (GPIO7)
- no-connect marks 0 -> 8
Changed lines of the file:
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@@
 		(color 0 0 0 0)
+	)
+	(no_connect
+		(at 165.1 114.3)
+	)
+	(no_connect
+		(at 165.1 88.9)
+	)
+	(no_connect
+		(at 119.38 86.36)
+	)
+	(no_connect
+		(at 119.38 83.82)
+	)
+	(no_connect
+		(at 165.1 116.84)
+	)
+	(no_connect
+		(at 165.1 106.68)
+	)
+	(no_connect
+		(at 137.16 60.96)
+	)
+	(no_connect
+		(at 119.38 76.2)
 	)
 	(wire
@@
 		)
 	)
-	(hierarchical_label "BTN 4"
+	(hierarchical_label "DI_IN"
 		(shape input)
-		(at 119.38 116.84 180)
+		(at 119.38 111.76 180)
+		(effects
+			(font
+				(size 1.27 1.27)
+			)
+			(justify right)
+		)
+	)
+	(hierarchical_label "BUZZER"
+		(shape output)
+		(at 165.1 101.6 0)
+		(effects
+			(font
+				(size 1.27 1.27)
+			)
+			(justify left)
+		)
+	)
+	(hierarchical_label "DI_PL"
+		(shape output)
+		(at 119.38 109.22 180)
+		(effects
+			(font
+				(size 1.27 1.27)
+			)
+			(justify right)
+		)
+	)
+	(hierarchical_label "REL_SAFE"
+		(shape output)
+		(at 119.38 101.6 180)
 		(effects
 			(font
@@
 		)
 	)
+	(hierarchical_label "EPD_CS"
+		(shape output)
+		(at 119.38 116.84 180)
+		(effects
+			(font
+				(size 1.27 1.27)
+			)
+			(justify right)
+		)
+	)
 	(hierarchical_label "ADC0"
 		(shape input)
@@
 		)
 	)
-	(hierarchical_label "BTN 2"
-		(shape input)
-		(at 119.38 111.76 180)
+	(hierarchical_label "L_G"
+		(shape output)
+		(at 119.38 96.52 180)
 		(effects
 			(font
@@
 		)
 	)
-	(hierarchical_label "RELAY"
-		(shape output)
-		(at 119.38 106.68 180)
+	(hierarchical_label "EPD_DC"
+		(shape output)
+		(at 119.38 119.38 180)
+		(effects
+			(font
+				(size 1.27 1.27)
+			)
+			(justify right)
+		)
+	)
+	(hierarchical_label "L_R"
+		(shape output)
+		(at 119.38 93.98 180)
 		(effects
 			(font
@@
 		)
 	)
+	(hierarchical_label "REL_ENLR"
+		(shape output)
+		(at 119.38 104.14 180)
+		(effects
+			(font
+				(size 1.27 1.27)
+			)
+			(justify right)
+		)
+	)
+	(hierarchical_label "L_B"
+		(shape output)
+		(at 119.38 99.06 180)
+		(effects
+			(font
+				(size 1.27 1.27)
+			)
+			(justify right)
+		)
+	)
 	(hierarchical_label "ENC 1B"
 		(shape output)
@@
 		)
 	)
-	(hierarchical_label "BTN 5"
-		(shape input)
-		(at 119.38 119.38 180)
-		(effects
-			(font
-				(size 1.27 1.27)
-			)
-			(justify right)
-		)
-	)
-	(hierarchical_label "BTN 3"
+	(hierarchical_label "EPD_BUSY"
 		(shape input)
 		(at 119.38 114.3 180)
@@
 		)
 	)
-	(hierarchical_label "BTN 1"
-		(shape input)
-		(at 119.38 109.22 180)
-		(effects
-			(font
-				(size 1.27 1.27)
-			)
-			(justify right)
-		)
-	)
-	(hierarchical_label "BTN 6"
-		(shape input)
+	(hierarchical_label "SPI SCK"
+		(shape output)
+		(at 165.1 91.44 0)
+		(effects
+			(font
+				(size 1.27 1.27)
+			)
+			(justify left)
+		)
+	)
+	(hierarchical_label "DI_CLK"
+		(shape output)
+		(at 119.38 106.68 180)
+		(effects
+			(font
+				(size 1.27 1.27)
+			)
+			(justify right)
+		)
+	)
+	(hierarchical_label "SPI TX"
+		(shape output)
+		(at 165.1 93.98 0)
+		(effects
+			(font
+				(size 1.27 1.27)
+			)
+			(justify left)
+		)
+	)
+	(hierarchical_label "SSD CS"
+		(shape output)
+		(at 165.1 96.52 0)
+		(effects
+			(font
+				(size 1.27 1.27)
+			)
+			(justify left)
+		)
+	)
+	(hierarchical_label "EPD_RES"
+		(shape output)
 		(at 119.38 121.92 180)
-		(effects
-			(font
-				(size 1.27 1.27)
-			)
-			(justify right)
-		)
-	)
-	(hierarchical_label "L_R"
-		(shape output)
-		(at 119.38 99.06 180)
-		(effects
-			(font
-				(size 1.27 1.27)
-			)
-			(justify right)
-		)
-	)
-	(hierarchical_label "SPI SCK"
-		(shape output)
-		(at 165.1 91.44 0)
-		(effects
-			(font
-				(size 1.27 1.27)
-			)
-			(justify left)
-		)
-	)
-	(hierarchical_label "L_G"
-		(shape output)
-		(at 119.38 101.6 180)
-		(effects
-			(font
-				(size 1.27 1.27)
-			)
-			(justify right)
-		)
-	)
-	(hierarchical_label "SPI TX"
-		(shape output)
-		(at 165.1 93.98 0)
-		(effects
-			(font
-				(size 1.27 1.27)
-			)
-			(justify left)
-		)
-	)
-	(hierarchical_label "SSD CS"
-		(shape output)
-		(at 165.1 96.52 0)
-		(effects
-			(font
-				(size 1.27 1.27)
-			)
-			(justify left)
-		)
-	)
-	(hierarchical_label "L_B"
-		(shape output)
-		(at 119.38 104.14 180)
 		(effects
 			(font
@@
 			)
 		)
-		(property "Footprint" "Module:RaspberryPi_Pico_Common_SMD"
+		(property "Footprint" "Module:RaspberryPi_Pico_SMD_HandSolder"
 			(at 142.24 146.05 0)
 			(effects
@@
 		(property "Description" "Versatile and inexpensive microcontroller module powered by RP2040 dual-core Arm Cortex-M0+ processor up to 133 MHz, 264kB SRAM, 2MB QSPI flash; also supports Raspberry Pi Pico 2"
 			(at 142.24 151.13 0)
-			(effects
-				(font
-					(size 1.27 1.27)
-				)
-				(hide yes)
-			)
-		)
-		(property "Placement" "Required"
-			(at 142.24 99.06 0)
 			(effects
 				(font
@@
 			)
 		)
-		(property "Footprint" "PCM_SparkFun-Jumper:Jumper_2_NC_Trace"
+		(property "Footprint" "Jumper:SolderJumper-2_P1.3mm_Bridged_Pad1.0x1.5mm"
 			(at 147.32 53.34 0)
 			(effects
@@
 		(property "Description" "Jumper, 2-pole, closed/bridged"
 			(at 147.32 53.34 0)
-			(effects
-				(font
-					(size 1.27 1.27)
-				)
-				(hide yes)
-			)
-		)
-		(property "Placement" "Required"
-			(at 147.32 53.34 90)
 			(effects
 				(font
@@
 			)
 		)
-		(property "Placement" "Required"
-			(at 147.32 46.99 90)
-			(effects
-				(font
-					(size 1.27 1.27)
-				)
-				(hide yes)
-			)
-		)
 		(pin "1"
 		)
@@
 			)
 		)
-		(property "Footprint" "PCM_SparkFun-Jumper:Jumper_2_NO"
+		(property "Footprint" "Jumper:SolderJumper-2_P1.3mm_Open_Pad1.0x1.5mm"
 			(at 114.3 78.74 0)
 			(effects
@@
 			(at 114.3 78.74 0)
 			(effects
-				(font
-					(size 1.27 1.27)
-				)
-				(hide yes)
-			)
-		)
-		(property "Placement" "Required"
-			(at 114.3 78.74 0)
-			(effects
