File: pcb/darkroom-timer/power_in.kicad_sch (KiCad schematic)
At the start: 5 parts, among them U2 L7805

Commit message: PCB Ready
Parts:
- added J6: Conn_01x02_Socket, TerminalBlock_Phoenix:TerminalBlock_Phoenix_MKDS-1,5-2_1x02_P5.00mm_Horizontal, symbol Connector:Conn_01x02_Socket
- added J7: Conn_01x03_Socket, TerminalBlock_Phoenix:TerminalBlock_Phoenix_MKDS-1,5-3_1x03_P5.00mm_Horizontal, symbol Connector:Conn_01x03_Socket
- C1: InvenTree Part # (none) -> 735; Placement Required -> (none)
- C2: value 0.33uF -> 0.1uF; InvenTree Part # (none) -> 735; Placement Required -> (none)
- TP1, TP2: Placement Required -> (none)
- U2: InvenTree Part # (none) -> 575; Placement Required -> (none)
Connections:
- net +24V: now also J6.2 (Pin_2)
- net GND renamed Earth
- net Earth: now also J6.1 (Pin_1), J7.3 (Pin_3)
- new net LINE: J7.2 (Pin_2)
- new net NEUT: J7.1 (Pin_1)

Commit message: Correct Connectors
Parts:
- J6: footprint TerminalBlock_Phoenix:TerminalBlock_Phoenix_MKDS-1,5-2_1x02_P5.00mm_Horizontal -> Connector_Phoenix_MC:PhoenixContact_MC_1,5_2-G-3.81_1x02_P3.81mm_Horizontal
Changed lines of the file:
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@@
 			)
 		)
-		(property "Footprint" "TerminalBlock_Phoenix:TerminalBlock_Phoenix_MKDS-1,5-2_1x02_P5.00mm_Horizontal"
+		(property "Footprint" "Connector_Phoenix_MC:PhoenixContact_MC_1,5_2-G-3.81_1x02_P3.81mm_Horizontal"
 			(at 115.57 95.25 0)
 			(effects
