File: pcb/darkroom-timer/rgb_output.kicad_sch (KiCad schematic)
At the start: 1 part, among them J2 Conn_01x06_Socket

Commit message: PCB Ready
Parts:
- J2: footprint (none) -> TerminalBlock_Phoenix:TerminalBlock_Phoenix_MKDS-1,5-6_1x06_P5.00mm_Horizontal; Placement Required -> (none)
Connections:
- net MOSFET 1/+L: now also J2.6 (Pin_6); no longer J2.1 (Pin_1)
- net MOSFET 1/-L: now also J2.5 (Pin_5); no longer J2.2 (Pin_2)
- net MOSFET 2/+L: now also J2.4 (Pin_4); no longer J2.3 (Pin_3)
- net MOSFET 2/-L: now also J2.3 (Pin_3); no longer J2.4 (Pin_4)
- net MOSFET 3/+L: now also J2.2 (Pin_2); no longer J2.5 (Pin_5)
- net MOSFET 3/-L: now also J2.1 (Pin_1); no longer J2.6 (Pin_6)
Changed lines of the file:
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@@
+	(wire
+		(pts
+			(xy 168.91 88.9) (xy 168.91 77.47)
+		)
+		(stroke
+			(width 0)
+			(type default)
+		)
+	)
 	(wire
 		(pts
 			(xy 166.37 80.01) (xy 166.37 91.44)
+		)
+		(stroke
+			(width 0)
+			(type default)
+		)
+	)
+	(wire
+		(pts
+			(xy 144.78 96.52) (xy 168.91 96.52)
 		)
 		(stroke
@@
 	(wire
 		(pts
-			(xy 166.37 91.44) (xy 168.91 91.44)
-		)
-		(stroke
-			(width 0)
-			(type default)
-		)
-	)
-	(wire
-		(pts
-			(xy 144.78 96.52) (xy 168.91 96.52)
+			(xy 166.37 99.06) (xy 168.91 99.06)
 		)
 		(stroke
@@
 	(wire
 		(pts
-			(xy 144.78 93.98) (xy 168.91 93.98)
+			(xy 166.37 91.44) (xy 168.91 91.44)
 		)
 		(stroke
@@
 	(wire
 		(pts
-			(xy 166.37 99.06) (xy 168.91 99.06)
-		)
-		(stroke
-			(width 0)
-			(type default)
-		)
-	)
-	(wire
-		(pts
-			(xy 168.91 88.9) (xy 168.91 77.47)
+			(xy 144.78 93.98) (xy 168.91 93.98)
 		)
 		(stroke
@@
 	(symbol
 		(lib_id "Connector:Conn_01x06_Socket")
-		(at 173.99 93.98 0)
+		(at 173.99 96.52 0)
+		(mirror x)
 		(unit 1)
 		(exclude_from_sim no)
@@
 		(on_board yes)
 		(dnp no)
-		(fields_autoplaced yes)
 		(property "Reference" "J2"
-			(at 175.26 93.9799 0)
+			(at 175.26 96.5201 0)
 			(effects
 				(font
@@
 		)
 		(property "Value" "Conn_01x06_Socket"
-			(at 175.26 96.5199 0)
+			(at 175.26 93.9801 0)
 			(effects
 				(font
@@
 			)
 		)
-		(property "Footprint" ""
-			(at 173.99 93.98 0)
+		(property "Footprint" "TerminalBlock_Phoenix:TerminalBlock_Phoenix_MKDS-1,5-6_1x06_P5.00mm_Horizontal"
+			(at 173.99 96.52 0)
 			(effects
 				(font
@@
 		)
 		(property "Datasheet" "~"
-			(at 173.99 93.98 0)
+			(at 173.99 96.52 0)
 			(effects
 				(font
@@
 		)
 		(property "Description" "Generic connector, single row, 01x06, script generated"
-			(at 173.99 93.98 0)
+			(at 173.99 96.52 0)
 			(effects
 				(font
-					(size 1.27 1.27)
-				)
-				(hide yes)
-			)
-		)
-		(property "Placement" "Required"
-			(at 173.99 93.98 0)
-			(effects
-				(font

Commit message: Correct Connectors
Parts:
- J2: footprint TerminalBlock_Phoenix:TerminalBlock_Phoenix_MKDS-1,5-6_1x06_P5.00mm_Horizontal -> Connector_Phoenix_MC:PhoenixContact_MC_1,5_6-G-3.81_1x06_P3.81mm_Horizontal
Changed lines of the file:
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@@
 			)
 		)
-		(property "Footprint" "TerminalBlock_Phoenix:TerminalBlock_Phoenix_MKDS-1,5-6_1x06_P5.00mm_Horizontal"
+		(property "Footprint" "Connector_Phoenix_MC:PhoenixContact_MC_1,5_6-G-3.81_1x06_P3.81mm_Horizontal"
 			(at 173.99 96.52 0)
 			(effects
