File: pcb/darkroom-timer/darkroom-timer.kicad_pcb (KiCad board)
At the start: 2 copper layers, 100 x 100 mm, 81 parts, among them J1 Micro_SD_Card_Det2, J2 Conn_01x06_Socket, J3 Conn_01x02_Socket, J4 EPD Connector, J5 Conn_01x02_Socket, J6 Conn_01x02_Socket, J7 Conn_01x03_Socket, K1 Relay_DPDT, K2 Relay_DPDT, Q1 BSS138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

Commit message: Correct Connectors
Parts:
- J2: footprint TerminalBlock_Phoenix:TerminalBlock_Phoenix_MKDS-1,5-6_1x06_P5.00mm_Horizontal -> Connector_Phoenix_MC:PhoenixContact_MC_1,5_6-G-3.81_1x06_P3.81mm_Horizontal
- J6: footprint TerminalBlock_Phoenix:TerminalBlock_Phoenix_MKDS-1,5-2_1x02_P5.00mm_Horizontal -> Connector_Phoenix_MC:PhoenixContact_MC_1,5_2-G-3.81_1x02_P3.81mm_Horizontal
- moved J6 9.78 mm to (138.8, 136.1)
- moved J2 5.76 mm to (125.0, 136.1)
Routing:
- net +24V: track 73.2 -> 79.7 mm
- net /RGB Output/MOSFET 3/PWR_NEG: track 12.4 -> 18.6 mm
- net Earth: track 16.7 -> 22.3 mm, vias 205 -> 206
- net /RGB Output/MOSFET 1/PWR_NEG: track 11.1 -> 9.20 mm

Commit message: Final PCB R0 design
Parts:
- added G***: LOGO, LOGO, F.Cu at (123.9, 57.4)
- added R30: 10k, Resistor_SMD:R_0805_2012Metric, B.Cu at (145.9, 86.2)
- added SW5: Start Switch, Button_Switch_THT:SW_PUSH_6mm_H13mm, F.Cu at (148.8, 83.8)
- J4: footprint Connector_IDC:IDC-Header_2x04_P2.54mm_Vertical -> Connector_PinHeader_2.54mm:PinHeader_2x04_P2.54mm_Vertical
- moved C6 3.60 mm to (159.1, 89.0)
- moved JP6 3.60 mm to (169.8, 83.5)
- moved TP7 3.60 mm to (162.6, 83.5)
- moved TP8 3.60 mm to (158.8, 83.5)
- moved TP9 3.60 mm to (166.4, 83.5)
- moved U5 3.60 mm to (162.6, 83.5)
- moved R27 3.18 mm to (157.6, 77.3)
Connections:
- C5 pad 1: +5V -> +3V3
- J4 pad 5: MOSI 5V -> MOSI 3V3
- J4 pad 6: SCK 5V -> SCK 3V3
- J4 pad 8: +5V -> +3V3
- U5 pad 12: unconnected-(U5-D1-Pad12) -> Net-(U5-D1)
Routing:
- net MOSI 3V3: track 67.6 -> 128.0 mm, vias 2 -> 4
- net SCK 3V3: track 69.5 -> 126.9 mm, vias 2 -> 4
- net MOSI 5V: track 83.5 -> 53.8 mm
- net Net-(U5-D1): track 0.00 -> 21.4 mm, vias 0 -> 2
- net +5V: track 340.0 -> 325.9 mm
- net +3.3V: track 242.7 -> 254.6 mm, vias 10 -> 9
- net SCK 5V: track 71.1 -> 60.3 mm
- net +3V3: track 0.00 -> 5.83 mm
- net /Digital Inputs/CLK: track 93.9 -> 99.3 mm
- net /Digital Inputs/PL: track 91.9 -> 96.9 mm, vias 3 -> 2
- net BTN 1: track 30.6 -> 27.9 mm
- net Net-(U4-Q7): track 47.1 -> 48.5 mm
- net /Digital Inputs/SER_OUT: track 59.8 -> 61.2 mm
- net /Logic Shifter 4/LV: track 33.2 -> 31.7 mm
- net Earth: vias 206 -> 210
Other:
- board text added: "Burn capitalism <3"
- board text added: "darkroom-timer R0 Copyright Frank Fourlas 2026"

Commit message: Settings page Major work + changes
Connections:
- C5 pad 1: +3V3 -> +3.3V
- J4 pad 8: +3V3 -> +3.3V
Routing:
- net +3.3V: track 254.6 -> 277.9 mm, vias 9 -> 10
- net +3V3: track 5.83 -> 0.00 mm
- net Earth: vias 210 -> 211
